Commit message: Rviz collegato (manca l'allineamento) + introdotto esempio di gestione robot tramite script python

File: src/robot_description/Cobotta.urdf (robot description, URDF)
Before this commit: robot Cobotta, 11 links, 10 joints
Links:
- link ROOT: geometry collision mesh filename=file:///home/marco/Desktop/charm_ws/src/robot_description/m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 scale=1.00000 1.00000 1.00000; visual mesh filename=file:///home/marco/Desktop/charm_ws/src/robot_description/m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 scale=1.00000 1.00000 1.00000
- link camera_link: geometry visual mesh filename=file:///home/marco/Desktop/charm_ws/src/robot_description/m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 scale=1.00000 1.00000 1.00000
- link link_gripper_l: geometry collision mesh filename=file:///home/marco/Desktop/charm_ws/src/robot_description/m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 scale=1.00000 1.00000 1.00000; visual mesh filename=file:///home/marco/Desktop/charm_ws/src/robot_description/m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 scale=1.00000 1.00000 1.00000
- link link_gripper_r: geometry collision mesh filename=file:///home/marco/Desktop/charm_ws/src/robot_description/m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 scale=1.00000 1.00000 1.00000; visual mesh filename=file:///home/marco/Desktop/charm_ws/src/robot_description/m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 scale=1.00000 1.00000 1.00000
- link link_j1: geometry collision mesh filename=file:///home/marco/Desktop/charm_ws/src/robot_description/m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 scale=1.00000 1.00000 1.00000; visual mesh filename=file:///home/marco/Desktop/charm_ws/src/robot_description/m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 scale=1.00000 1.00000 1.00000
- link link_j2: geometry collision mesh filename=file:///home/marco/Desktop/charm_ws/src/robot_description/m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 scale=1.00000 1.00000 1.00000; visual mesh filename=file:///home/marco/Desktop/charm_ws/src/robot_description/m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 scale=1.00000 1.00000 1.00000
- link link_j3: geometry collision mesh filename=file:///home/marco/Desktop/charm_ws/src/robot_description/m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 scale=1.00000 1.00000 1.00000; visual mesh filename=file:///home/marco/Desktop/charm_ws/src/robot_description/m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 scale=1.00000 1.00000 1.00000
- link link_j4: geometry collision mesh filename=file:///home/marco/Desktop/charm_ws/src/robot_description/m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 scale=1.00000 1.00000 1.00000; visual mesh filename=file:///home/marco/Desktop/charm_ws/src/robot_description/m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 scale=1.00000 1.00000 1.00000
- link link_j5: geometry collision mesh filename=file:///home/marco/Desktop/charm_ws/src/robot_description/m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 scale=1.00000 1.00000 1.00000; visual mesh filename=file:///home/marco/Desktop/charm_ws/src/robot_description/m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 scale=1.00000 1.00000 1.00000
- link link_j6: geometry collision mesh filename=file:///home/marco/Desktop/charm_ws/src/robot_description/m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 scale=1.00000 1.00000 1.00000; visual mesh filename=file:///home/marco/Desktop/charm_ws/src/robot_description/m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 scale=1.00000 1.00000 1.00000
Joints:
- joint joint3: limit lower=0.00000 upper=0.00000 effort=0.00000 velocity=5.00000 -> lower=0.314159 upper=2.443460 effort=100.00000 velocity=1.66187

Commit message: Allineamento tra Gazebo e RViz attuato - modifica al file urdf- joint 3 posizione e asse - joint 5 asse

File: src/robot_description/Cobotta.urdf (robot description, URDF)
Before this commit: robot Cobotta, 11 links, 10 joints
Joints:
- joint joint3: axis 0.00000 0.00000 1.00000 -> 0.00000 0.00000 -1.00000; origin xyz=-0.16500 0.00000 0.00000 rpy=3.14159 -0.00000 3.14159 -> xyz=-0.16500 0.00000 0.00000 rpy=3.14159 -0.00000 1.5708
- joint joint5: axis 0.00000 0.00000 1.00000 -> 0.00000 0.00000 -1.00000

Commit message: Aggiunta piatto e script per prenderlo

File: src/robot_description/Cobotta.urdf (robot description, URDF)
Before this commit: robot Cobotta, 11 links, 10 joints
Links:
- link ROOT: geometry collision mesh filename=file:///home/nicolas/Scrivania/charm_ws/src/robot_descripti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 scale=1.00000 1.00000 1.00000; visual mesh filename=file:///home/nicolas/Scrivania/charm_ws/src/robot_descripti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 scale=1.00000 1.00000 1.00000
- link camera_link: geometry visual mesh filename=file:///home/nicolas/Scrivania/charm_ws/src/robot_descripti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 scale=1.00000 1.00000 1.00000
- link link_gripper_l: geometry collision mesh filename=file:///home/nicolas/Scrivania/charm_ws/src/robot_descripti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 scale=1.00000 1.00000 1.00000; visual mesh filename=file:///home/nicolas/Scrivania/charm_ws/src/robot_descripti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 scale=1.00000 1.00000 1.00000
- link link_gripper_r: geometry collision mesh filename=file:///home/nicolas/Scrivania/charm_ws/src/robot_descripti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 scale=1.00000 1.00000 1.00000; visual mesh filename=file:///home/nicolas/Scrivania/charm_ws/src/robot_descripti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 scale=1.00000 1.00000 1.00000
- link link_j1: geometry collision mesh filename=file:///home/nicolas/Scrivania/charm_ws/src/robot_descripti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 scale=1.00000 1.00000 1.00000; visual mesh filename=file:///home/nicolas/Scrivania/charm_ws/src/robot_descripti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 scale=1.00000 1.00000 1.00000
- link link_j2: geometry collision mesh filename=file:///home/nicolas/Scrivania/charm_ws/src/robot_descripti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 scale=1.00000 1.00000 1.00000; visual mesh filename=file:///home/nicolas/Scrivania/charm_ws/src/robot_descripti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 scale=1.00000 1.00000 1.00000
- link link_j3: geometry collision mesh filename=file:///home/nicolas/Scrivania/charm_ws/src/robot_descripti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 scale=1.00000 1.00000 1.00000; visual mesh filename=file:///home/nicolas/Scrivania/charm_ws/src/robot_descripti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 scale=1.00000 1.00000 1.00000
- link link_j4: geometry collision mesh filename=file:///home/nicolas/Scrivania/charm_ws/src/robot_descripti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 scale=1.00000 1.00000 1.00000; visual mesh filename=file:///home/nicolas/Scrivania/charm_ws/src/robot_descripti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 scale=1.00000 1.00000 1.00000
- link link_j5: geometry collision mesh filename=file:///home/nicolas/Scrivania/charm_ws/src/robot_descripti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 scale=1.00000 1.00000 1.00000; visual mesh filename=file:///home/nicolas/Scrivania/charm_ws/src/robot_descripti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 scale=1.00000 1.00000 1.00000
- link link_j6: geometry collision mesh filename=file:///home/nicolas/Scrivania/charm_ws/src/robot_descripti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 scale=1.00000 1.00000 1.00000; visual mesh filename=file:///home/nicolas/Scrivania/charm_ws/src/robot_descripti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 scale=1.00000 1.00000 1.00000

Commit message: Eliminato il plain di simulazione gesto + corretta posizione di monitoring

File: src/robot_description/Cobotta.urdf (robot description, URDF)
Before this commit: robot Cobotta, 11 links, 10 joints
Links:
- link ROOT: geometry collision mesh filename=file:///home/marco/Desktop/charm_ws/src/robot_description/m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 scale=1.00000 1.00000 1.00000; visual mesh filename=file:///home/marco/Desktop/charm_ws/src/robot_description/m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 scale=1.00000 1.00000 1.00000
- link camera_link: geometry visual mesh filename=file:///home/marco/Desktop/charm_ws/src/robot_description/m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 scale=1.00000 1.00000 1.00000
- link link_gripper_l: geometry collision mesh filename=file:///home/marco/Desktop/charm_ws/src/robot_description/m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 scale=1.00000 1.00000 1.00000; visual mesh filename=file:///home/marco/Desktop/charm_ws/src/robot_description/m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 scale=1.00000 1.00000 1.00000
- link link_gripper_r: geometry collision mesh filename=file:///home/marco/Desktop/charm_ws/src/robot_description/m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 scale=1.00000 1.00000 1.00000; visual mesh filename=file:///home/marco/Desktop/charm_ws/src/robot_description/m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 scale=1.00000 1.00000 1.00000
- link link_j1: geometry collision mesh filename=file:///home/marco/Desktop/charm_ws/src/robot_description/m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 scale=1.00000 1.00000 1.00000; visual mesh filename=file:///home/marco/Desktop/charm_ws/src/robot_description/m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 scale=1.00000 1.00000 1.00000
- link link_j2: geometry collision mesh filename=file:///home/marco/Desktop/charm_ws/src/robot_description/m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 scale=1.00000 1.00000 1.00000; visual mesh filename=file:///home/marco/Desktop/charm_ws/src/robot_description/m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 scale=1.00000 1.00000 1.00000
- link link_j3: geometry collision mesh filename=file:///home/marco/Desktop/charm_ws/src/robot_description/m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 scale=1.00000 1.00000 1.00000; visual mesh filename=file:///home/marco/Desktop/charm_ws/src/robot_description/m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 scale=1.00000 1.00000 1.00000
- link link_j4: geometry collision mesh filename=file:///home/marco/Desktop/charm_ws/src/robot_description/m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 scale=1.00000 1.00000 1.00000; visual mesh filename=file:///home/marco/Desktop/charm_ws/src/robot_description/m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 scale=1.00000 1.00000 1.00000
- link link_j5: geometry collision mesh filename=file:///home/marco/Desktop/charm_ws/src/robot_description/m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 scale=1.00000 1.00000 1.00000; visual mesh filename=file:///home/marco/Desktop/charm_ws/src/robot_description/m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 scale=1.00000 1.00000 1.00000
- link link_j6: geometry collision mesh filename=file:///home/marco/Desktop/charm_ws/src/robot_description/m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 scale=1.00000 1.00000 1.00000; visual mesh filename=file:///home/marco/Desktop/charm_ws/src/robot_description/m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 scale=1.00000 1.00000 1.00000
